File: Hardware-Electronics/module/Flight-Controller/drone-v0/drone-v0.kicad_sch (KiCad schematic)
At the start: 11 parts, among them IC1 REG1117-3.3, IC2 CP2102N-A02-GQFN28, J1 2171790001, U1 ESP32-S3-MINI-1U-N8

Commit message: Added Auto Programmer
Parts:
- added C3, C6: 0.1uF, CAPC1608X90N, symbol Ceramic Cap 0.1uF 0603:06035C104JAZ2A
- added C4, C5: 4.7uF, CAPC1608X90N, symbol Ceramic Cap 4.7uF 0603:CGA3E1X5R0J475K080AC
- added IC3: SBC846BDW1T1G, SOT65P210X110-6N, symbol SBC846BDW1T1G:SBC846BDW1T1G
- added R4, R5: 10k, RESC1608X50N, symbol Res 10k 0603:CRCW060310K0FKEI
Connections:
- net 3V3: now also C5.1, C6.1
- net GND: now also IC2.29 (BGND), C3.2, C4.2, C5.2, C6.2
- net VBUS: now also IC2.7 (VREGIN), IC2.8 (VBUS), C3.1, C4.1
- net RTS: now reaches IC2.24 (RTS)
- net RTS: now also IC3.1 (E1), R5.2
- net U0TXD: now reaches IC2.25 (RXD)
- net U0RXD: now reaches IC2.26 (TXD)
- net DTS: now reaches IC2.28 (DTR)
- net DTS: now also IC3.4 (E2), R4.1
- new net: IC3.2 (B1), R4.2
- new net: IC3.5 (B2), R5.1
- new net CHIP_PU: IC3.3 (C1)
- new net GPIO0: IC3.6 (C2)
- no-connect marks 6 -> 22
Other:
- note added: "Auto Programmer"
- moved on the sheet: IC2, U1

Commit message: Added: Sensors, Espressif Schematic file and Boot Options
Parts:
- removed R2: 5.1k, RESC1608X55N, symbol Res 5.1k 0603:CR0603-FX-5101ELF
- added C10, C7, C9: 0.1uF, CAPC1608X90N, symbol Ceramic Cap 0.1uF 0603:06035C104JAZ2A
- added C8: 10uF, CAPC1608X90N, symbol Ceramic Cap 10uF 0603:C1608X7R1A106M080AT
- added IC4: ICM-20602, IAM20680HP, symbol ICM-20602:ICM-20602
- added LED2: 150060RS83000, LEDC1608X115N, symbol Red LED 0603:150060RS83000
- added R2, R7: 1k, RESC1608X50N, symbol Res 1k 0603:CRCW06031K00FKEI
- added R6: 10k, RESC1608X50N, symbol Res 10k 0603:CRCW060310K0FKEI
- added S1, S2: TL3301AF160QG, TL3301AF160QG, symbol Tactile switch:TL3301AF160QG
Connections:
- net 3V3: now also U1.3 (3V3), C7.2, C8.2, R6.2, R7.1
- net D+: no longer D1.1 (I/O_1), J1.A6 (DP1), J1.B7 (DN2)
- net D-: no longer D1.2 (I/O_2), J1.A7 (DN1), J1.B6 (DP2)
- net GND: now also C10.1, C7.1, C8.1, C9.1, LED2.1 (K), S1.1 (COM_1), S1.2 (COM_2), S2.1 (COM_1), S2.2 (COM_2)
- net GPIO0: now also U1.4 (IO0), C10.2, S2.3 (NO_1), S2.4 (NO_2)
- net VBUS: no longer J1.A4B9 (VBUS1), J1.B4A9 (VBUS2)
- net ESP_EN: now reaches U1.45 (EN)
- net ESP_EN: now also C9.2, R6.1, S1.3 (NO_1), S1.4 (NO_2)
- net at LED1.2 (A): now also R7.2
- net RX_D0: no longer names the net of U1.40 (RXD0)
- net TX_D0: no longer names the net of U1.39 (TXD0)
- new net: LED2.2 (A), R2.2
- new net 5V: R2.1
- new net 5V_USB: J1.A4B9 (VBUS1), J1.B4A9 (VBUS2)
- new net USB_N: D1.2 (I/O_2), J1.A7 (DN1), J1.B7 (DN2)
- new net USB_P: D1.1 (I/O_1), J1.A6 (DP1), J1.B6 (DP2)
Other:
- note added: "BOOT"
- note added: "DECOUPLING"
- note added: "Debugging LED"
- note added: "IMU - Sensor"
- note added: "RESET"
- moved on the sheet: LED1, U1

Commit message: Added: - New PCB Design - Completed ESP32 configuration comp. - Ran Electrical Rules Check (ERC)
Parts:
- removed D1: D3V3XA4B10LP-7, D3V3XA4B10LP7, symbol D3V3XA4B10LP-7:D3V3XA4B10LP-7
- removed IC4: ICM-20602, IAM20680HP, symbol ICM-20602:ICM-20602
- removed J1: 2171790001, 2171790001:MOLEX_2171790001, symbol 217179-0001:2171790001
- removed R1, R3: 5.1k, RESC1608X55N, symbol Res 5.1k 0603:CR0603-FX-5101ELF
- added J2: USB_C_Receptacle_USB2.0_16P, 2171790001(1):MOLEX_2171790001, symbol Connector:USB_C_Receptacle_USB2.0_16P
- added R1, R3: 5.1k, Res 5.1k 0603:RESC1608X55N, symbol Device:R
- added U2: D3V3XA4B10LP, Package_DFN_QFN:Diodes_UDFN-10_1.0x2.5mm_P0.5mm, symbol Power_Protection:D3V3XA4B10LP
- C1: footprint 298D106X0010M2T -> Cap 10uF 0603:CAPC1608X90N
- C10, C2, C3, C6, C7, C9: footprint CAPC1608X90N -> Cap 0.1uF 0603:CAPC1608X90N
- C4, C5: footprint CAPC1608X90N -> Cap 4.7uF 0603:CAPC1608X90N
- C8: footprint CAPC1608X90N -> Cap 10uF 0603:CAPC1608X90N
- IC1: footprint SOT230P700X180-4N -> REG1117-3.3:SOT230P700X180-4N
- IC2: footprint QFN50P500X500X80-29N-D -> CP2102N-A02-GQFN28:QFN50P500X500X80-29N-D
- IC3: footprint SOT65P210X110-6N -> Res 10k 0603:RESC1608X50N
- LED1, LED2: footprint LEDC1608X115N -> Red LED 0603:LEDC1608X115N
- R2, R7: footprint RESC1608X50N -> Res 1k 0603:RESC1608X50N
- R4, R5, R6: footprint RESC1608X50N -> Res 10k 0603:RESC1608X50N
- S1, S2: footprint TL3301AF160QG -> TL3301AF160QG:TL3301AF160QG
Connections:
- net CHIP_PU is gone; now on net ESP_EN: IC3.3 (C1)
- net D+ is gone; now on net USB_P: IC2.4 (D+)
- net D- is gone; now on net USB_N: IC2.5 (D-)
- net U0RXD is gone; now on net USB_RX: IC2.26 (TXD)
- net U0TXD is gone; now on net USB_TX: IC2.25 (RXD)
- net GND: now also J2.A1 (GND), J2.A12 (GND), J2.B1 (GND), J2.B12 (GND), J2.S1 (SHIELD), R1.2, R3.2, U2.3 (VSS), U2.8 (VSS)
- net USB_N: now also J2.A7 (D-), J2.B7 (D-), U2.2
- net USB_P: now also J2.A6 (D+), J2.B6 (D+), U2.1
- net USB_TX: now reaches U1.39 (TXD0)
- net USB_RX: now reaches U1.40 (RXD0)
- net 3V3 renamed +3V3
- net +3V3: now also IC2.7 (VREGIN)
- net 5V renamed +5V_USB
- net +5V_USB: now also C2.2, C3.1, C4.1, IC1.3 (VIN), IC2.8 (VBUS), J2.A4 (VBUS), J2.A9 (VBUS), J2.B4 (VBUS), J2.B9 (VBUS), U2.4
- removed net VBUS: C2.2, C3.1, C4.1, IC1.3 (VIN), IC2.7 (VREGIN), IC2.8 (VBUS)
- new net: J2.B5 (CC2), R1.1
- new net: J2.A5 (CC1), R3.1
- no-connect marks 22 -> 61
Other:
- note added: "ESP32-S3-MINI-1U-N8"
- note added: "Flight Controler V0"
- note removed: "IMU - Sensor"
- moved on the sheet: C1, C10, C2, C3, C4, C5, C6, C7, C8, C9, IC1, IC2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

Commit message: Updates: dual LDO power design for STM32F405 flight controller - Added 3V3_MCU and 3V3_SNS rails for noise isolation - Integrated USB-C power input and SWD header - Finalized ESC, IMU, and barometer connections - Verified power sequencing and decoupling networks
Parts:
- removed C1: 10uF, Cap 10uF 0603:CAPC1608X90N, symbol Tant Cap 10uF 0603:298D106X0010M2T
- removed C10, C3, C6, C7, C9: 0.1uF, Cap 0.1uF 0603:CAPC1608X90N, symbol Ceramic Cap 0.1uF 0603:06035C104JAZ2A
- removed C2: 10uF, Cap 0.1uF 0603:CAPC1608X90N, symbol Ceramic Cap 10uF 0603:C1608X7R1A106M080AT
- removed C4, C5: 4.7uF, Cap 4.7uF 0603:CAPC1608X90N, symbol Ceramic Cap 4.7uF 0603:CGA3E1X5R0J475K080AC
- removed C8: 10uF, Cap 10uF 0603:CAPC1608X90N, symbol Ceramic Cap 10uF 0603:C1608X7R1A106M080AT
- removed IC1: REG1117-3.3, REG1117-3.3:SOT230P700X180-4N, symbol REG1117-3.3:REG1117-3.3
- removed IC2: CP2102N-A02-GQFN28, CP2102N-A02-GQFN28:QFN50P500X500X80-29N-D, symbol CP2102N-A02-GQFN28:CP2102N-A02-GQFN28
- removed IC3: SBC846BDW1T1G, Res 10k 0603:RESC1608X50N, symbol SBC846BDW1T1G:SBC846BDW1T1G
- removed J2: USB_C_Receptacle_USB2.0_16P, 2171790001(1):MOLEX_2171790001, symbol Connector:USB_C_Receptacle_USB2.0_16P
- removed LED1, LED2: 150060RS83000, Red LED 0603:LEDC1608X115N, symbol Red LED 0603:150060RS83000
- removed R2, R7: 1k, Res 1k 0603:RESC1608X50N, symbol Res 1k 0603:CRCW06031K00FKEI
- removed R4, R5, R6: 10k, Res 10k 0603:RESC1608X50N, symbol Res 10k 0603:CRCW060310K0FKEI
- removed S1, S2: TL3301AF160QG, TL3301AF160QG:TL3301AF160QG, symbol Tactile switch:TL3301AF160QG
- removed U1: ESP32-S3-MINI-1U-N8, ESP32-S3-MINI-1U-N8:XCVR_ESP32-S3-MINI-1U-N8, symbol ESP32-S3-MINI-1U-N8:ESP32-S3-MINI-1U-N8
- removed U2: D3V3XA4B10LP, Package_DFN_QFN:Diodes_UDFN-10_1.0x2.5mm_P0.5mm, symbol Power_Protection:D3V3XA4B10LP
- added C1, C11: 2.2uF, symbol Device:C
- added C10, C14, C2: 1uF, symbol Device:C
- added C19, C25, C26, C31: 2u2, symbol Device:C
- added C20, C21, C22, C23, C24, C30, C4: 100n, symbol Device:C
- added C27, C28, C7: 10p, symbol Device:C
- added C29, C6: 10n, symbol Device:C
- added C3: 0.1uF, symbol Device:C
- added C5: 4u7, symbol Device:C
- added C8: 1u, symbol Device:C
- added C9: C, symbol Device:C
- added D1: PMEG4010BEA,115, PMEG4010BEA,:SOD2512X110N, symbol PMEG4010BEA,:PMEG4010BEA,115
- added IC1: MS561101BA03-50, MS561101BA03-50, symbol MS561101BA03-50:MS561101BA03-50
- added J1: USB_C_Receptacle_USB2.0_16P, 2171790001(1):MOLEX_2171790001, symbol Connector:USB_C_Receptacle_USB2.0_16P
- added J2: 53254-0470, 532540470, symbol 53254-0470:53254-0470
- added J3: Conn_ARM_JTAG_SWD_10, symbol Connector:Conn_ARM_JTAG_SWD_10
- added L1: L, symbol Device:L
- added LED1, LED2, LED3, LED4: SML-P11UTT86R, KDZLV100, symbol RED LED 0402:SML-P11UTT86R
- added R10: 18.2k, symbol Device:R
- added R11, R16, R17: 100k, symbol Device:R
- added R12: 182k, symbol Device:R
- added R13: 1M, symbol Device:R
- added R14, R15, R7, R8: 1k, symbol Device:R
- added R2: 5.1k, symbol Device:R
- added R4, R6, R9: 10k, symbol Device:R
- added R5: 0R, symbol Device:R
- added SW1: PTS810 SJK 250 SMTR LFS, PTS810_CNK, symbol PTS810SJK250SMTR LFS:PTS810_SJK_250_SMTR_LFS
- added U1, U6: TLV76733DRVR, TLV76733DRVR:DRV0006A-IPC_B, symbol TLV76733DRVR:TLV76733DRVR
- added U2: ICM-42688-P, ICM-42688-P:PQFN50P300X250X97-14N, symbol ICM-42688-P:ICM-42688-P
- added U3: STM32F405RGTx, Package_QFP:LQFP-64_10x10mm_P0.5mm, symbol MCU_ST_STM32F4:STM32F405RGTx
- added U4: NUF2042XV6T1G, NUF2042XV6T1G:SON_2XV6T1G_ONS, symbol Power_Protection:USBLC6-2SC6
- added U5: LT8609SIV_TRPBF, LT8609SIV_TRPBF:REG_LT8609SIV_TRPBF, symbol LT8609SIV:LT8609SIV_TRPBF
- added Y1: Crystal, ECS-400-10-37B2-CKM-TR:ECS4001037B2CKMTR, symbol Device:Crystal
- R1: footprint Res 5.1k 0603:RESC1608X55N -> (none)
- R3: value 5.1k -> 10k; footprint Res 5.1k 0603:RESC1608X55N -> (none)
Connections:
- net GND: now also C1.2, C10.2, C11.2, C14.2, C19.2, C2.2, C20.2, C21.2, C22.2, C23.2, C24.2, C25.2, C26.2, C27.2, C28.2, C29.2, C3.2, C30.2, C31.2, C4.2, C5.2, C6.2, C8.2, C9.2, IC1.3 (GND), IC1.4 (CSB_1), IC1.5 (CSB_2), J1.A1 (GND), J1.A12 (GND), J1.B1 (GND), J1.B12 (GND), J1.S1 (SHIELD), J2.1, J3.3 (GND), J3.5 (GND), J3.9 (GNDDetect), R10.2, R12.2, R14.2, R15.2, R17.2, R2.2, R4.2, R7.2, R8.2, U1.3 (GND), U1.5 (GND), U1.7 (Pad), U2.11 (RESV_11), U2.6 (GND), U2.7 (RESV_7), U2.9 (INT2/FSYNC/CLKIN), U3.12 (VSSA), U3.18 (VSS), U3.63 (VSS), U4.2 (GND), U5.14 (GND), U5.17 (GND), U5.3 (GND), U5.4 (GND), U5.8 (GND), U6.3 (GND), U6.5 (GND), U6.7 (Pad); no longer R3.2
- net at R1.1: now also J1.B5 (CC2)
- net 3V3_MCU: now reaches R3.1
- net 3V3_MCU: now also C1.1, C19.1, C20.1, C21.1, C22.1, C23.1, C24.1, J3.1 (VTref), LED4. (A), R16.1, R6.1, R9.1, SW1.1, SW1.2, U1.1 (OUT), U1.2 (SNS), U3.1 (VBAT), U3.13 (VDDA), U3.19 (VDD), U3.32 (VDD), U3.48 (VDD), U3.64 (VDD)
- new net: C7.1, R12.1, R13.2, U5.13 (FB)
- new net: C28.1, R5.1, Y1.2
- new net: LED3. (A), R14.1
- new net: LED2. (A), R8.1
- new net: L1.1, U5.5 (SW), U5.6 (SW)
- new net: J1.A5 (CC1), R2.1
- new net: C6.1, U5.15 (TR/SS)
- new net: R11.2, U5.12 (PG)
- new net: R10.1, U5.1 (RT)
- new net: C8.1, U5.2 (INTVCC)
- new net: U5.7 (N/C), U5.NC1 (N/C), U5.NC2 (N/C), U5.NC3 (N/C), U5.NC4 (N/C)
- new net: LED1. (A), R7.1
- new net: LED4. (A), R15.1
- new net +5V: C10.1, C2.1, C7.2, C9.1, D1.1 (K), J2.4, L1.2, LED1. (A), R11.1, R13.1, U1.4 (EN), U1.6 (IN), U4.5 (VBUS), U6.4 (EN), U6.6 (IN)
- new net 3V3_SNS: C11.1, C29.1, C30.1, C31.1, C4.1, IC1.1 (VDD), IC1.2 (PS), LED2. (A), U2.4 (INT1/INT), U2.5 (VDDIO), U2.8 (VDD), U6.1 (OUT), U6.2 (SNS)
- new net BOOT0: R4.1, SW1.3, SW1.4, U3.60 (BOOT0)
- new net CURR_IN: U3.8 (PC0)
- new net D+: J1.A6 (D+), J1.B6 (D+), U3.45 (PA12), U4.3 (I/O2), U4.4 (I/O2)
- new net D-: J1.A7 (D-), J1.B7 (D-), U3.44 (PA11), U4.1 (I/O1), U4.6 (I/O1)
- new net ESC_TLM: U3.53 (PC12)
- new net I2C2_SCL: R3.2, U3.29 (PB10)
- new net I2C2_SDA: R6.2, U3.30 (PB11)
- new net M1: U3.37 (PC6)
- new net M2: U3.38 (PC7)
- new net M3: U3.26 (PB0)
- new net M4: U3.27 (PB1)
- new net NRST: C14.1, J3.10 (~{RESET}), R9.2
- new net NRTS: U3.7 (NRST)
- new net OSC_IN: C27.1, U3.5 (PH0), Y1.1
- new net OSC_OUT: R5.2, U3.6 (PH1)
- new net SCL: IC1.8 (SCLK)
- new net SDA: IC1.7 (SDI/SDA)
- new net SPI1_MISO: U2.1 (AP_SDO/AP_AD0), U3.22 (PA6)
- new net SPI1_MOSI: U2.14 (AP_SDA/AP_SDIO/AP_SDI), U3.23 (PA7)
- new net SPI1_NSS: U2.12 (AP_CS), U3.20 (PA4)
- new net SPI1_SCK: U2.13 (AP_SCL/AP_SCLK), U3.21 (PA5)
- new net SWCLK: J3.4 (SWCLK/TCK), R17.1, U3.49 (PA14)
- new net SWDIO: J3.2 (SWDIO/TMS), R16.2, U3.46 (PA13)
- new net SWO: J3.6 (SWO/TDO), U3.55 (PB3)
- new net UART4_RX: J2.3, U3.15 (PA1)
- new net UART4_TX: J2.2, U3.14 (PA0)
- new net VBAT: C5.1, LED3. (A), U5.10 (VIN), U5.11 (EN/UV), U5.9 (VIN)
- new net VBUS: C3.1, D1.2 (A), J1.A4 (VBUS), J1.A9 (VBUS), J1.B4 (VBUS), J1.B9 (VBUS)
- new net VCAP1: C25.1, U3.31 (VCAP_1)
- new net VCAP2: C26.1, U3.47 (VCAP_2)
- no-connect marks 61 -> 6
Other:
- note added: "Antenna Connector"
- note added: "BUTTONS"
- note added: "Barometer Sensor"
- note added: "Connector"
- note added: "Crystal Oscillator"
- note added: "Current Signal"
- note added: "DSHOT"
- note added: "Decoupling capacitor bank MCU"
- note added: "ESC Connector"
- note added: "GND"
- note added: "IMU 6-Axis Sensor"
- note added: "JTAG - connector"
- note added: "LDO - Voltage Regulator MCU"
- note added: "LDO - Voltage Regulator Sensor"
- note added: "LED Debugger"
- note added: "Power"
- note added: "STM32F405"
- note added: "Sensor"
- note added: "Step-Down Regulator"
- note added: "Telemetry (UART TX)"
- note added: "USB C + ESD Protection"
- note added: "Vbat"
- note removed: "Auto Programmer"
- note removed: "BOOT"
- note removed: "DECOUPLING"
- note removed: "Debugging LED"
- note removed: "ESD Protection"
- note removed: "ESP32-S3-MINI-1U-N8"
- note removed: "LDO"
- note removed: "RESET"
- note removed: "USB Type-C"
- note removed: "USB-UART Bridge"

Commit message: Added: STM32 Try resolve with rebase
Parts:
- removed C10: 1uF, symbol Device:C
- removed C11: 2.2uF, symbol Device:C
- removed LED4: SML-P11UTT86R, KDZLV100, symbol RED LED 0402:SML-P11UTT86R
- removed R15: 1k, symbol Device:R
- removed U6: TLV76733DRVR, TLV76733DRVR:DRV0006A-IPC_B, symbol TLV76733DRVR:TLV76733DRVR
- added J4: SM08B-SRSS-TB, SM08B-SRSS-TB:JST_SM08B-SRSS-TB, symbol SM08B-SRSS-TB:SM08B-SRSS-TB
- C9: value C -> 22u
- J3: footprint (none) -> FTSH-105-01-F-DH:FTSH-105-XX-YYY-DH
- L1: value L -> 2u2
Connections:
- net 3V3_SNS is gone; now on net +3V3: C29.1, C30.1, C31.1, C4.1, IC1.1 (VDD), IC1.2 (PS), LED2. (A), U2.4 (INT1/INT), U2.5 (VDDIO), U2.8 (VDD)
- net CURR_IN: now also J4.2
- net ESC_TLM: now also J4.1
- net GND: now also J4.8
- net M1: now also J4.6
- net M2: now also J4.5
- net M3: now also J4.4
- net M4: now also J4.3
- net 3V3_MCU renamed +3V3
- new net Vbat: J4.7
Other:
- note removed: "LDO - Voltage Regulator Sensor"

Commit message: Apply .gitignore
Parts:
- added LED4: SML-P11UTT86R, KDZLV100, symbol RED LED 0402:SML-P11UTT86R
- added R15: 1k, symbol Device:R
Connections:
- net GND: now also R15.2
- net LED_OUT: now reaches U3.9 (PC1)
- net LED_OUT: now also LED4. (A)
- new net: LED4. (A), R15.1
