File: Hardware-Electronics/module/Flight-Controller/drone-v0/drone-v0.kicad_sch (KiCad schematic)
At the start: 27 parts, among them IC1 REG1117-3.3, IC2 CP2102N-A02-GQFN28, IC3 SBC846BDW1T1G, J2 USB_C_Receptacle_USB2.0_16P, U1 ESP32-S3-MINI-1U-N8, U2 D3V3XA4B10LP

Commit message: Flight Controller updates (rebased) (#20)
* Updates: dual LDO power design for STM32F405 flight controller
- Added 3V3_MCU and 3V3_SNS rails for noise isolation
- Integrated USB-C power input and SWD header
- Finalized ESC, IMU, and barometer connections
- Verified power sequencing and decoupling networks

* Added: STM32 Try resolve with rebase

* Apply .gitignore
Parts:
- removed C1: 10uF, Cap 10uF 0603:CAPC1608X90N, symbol Tant Cap 10uF 0603:298D106X0010M2T
- removed C10, C3, C6, C7, C9: 0.1uF, Cap 0.1uF 0603:CAPC1608X90N, symbol Ceramic Cap 0.1uF 0603:06035C104JAZ2A
- removed C2: 10uF, Cap 0.1uF 0603:CAPC1608X90N, symbol Ceramic Cap 10uF 0603:C1608X7R1A106M080AT
- removed C4, C5: 4.7uF, Cap 4.7uF 0603:CAPC1608X90N, symbol Ceramic Cap 4.7uF 0603:CGA3E1X5R0J475K080AC
- removed C8: 10uF, Cap 10uF 0603:CAPC1608X90N, symbol Ceramic Cap 10uF 0603:C1608X7R1A106M080AT
- removed IC1: REG1117-3.3, REG1117-3.3:SOT230P700X180-4N, symbol REG1117-3.3:REG1117-3.3
- removed IC2: CP2102N-A02-GQFN28, CP2102N-A02-GQFN28:QFN50P500X500X80-29N-D, symbol CP2102N-A02-GQFN28:CP2102N-A02-GQFN28
- removed IC3: SBC846BDW1T1G, Res 10k 0603:RESC1608X50N, symbol SBC846BDW1T1G:SBC846BDW1T1G
- removed J2: USB_C_Receptacle_USB2.0_16P, 2171790001(1):MOLEX_2171790001, symbol Connector:USB_C_Receptacle_USB2.0_16P
- removed LED1, LED2: 150060RS83000, Red LED 0603:LEDC1608X115N, symbol Red LED 0603:150060RS83000
- removed R2, R7: 1k, Res 1k 0603:RESC1608X50N, symbol Res 1k 0603:CRCW06031K00FKEI
- removed R4, R5, R6: 10k, Res 10k 0603:RESC1608X50N, symbol Res 10k 0603:CRCW060310K0FKEI
- removed S1, S2: TL3301AF160QG, TL3301AF160QG:TL3301AF160QG, symbol Tactile switch:TL3301AF160QG
- removed U1: ESP32-S3-MINI-1U-N8, ESP32-S3-MINI-1U-N8:XCVR_ESP32-S3-MINI-1U-N8, symbol ESP32-S3-MINI-1U-N8:ESP32-S3-MINI-1U-N8
- removed U2: D3V3XA4B10LP, Package_DFN_QFN:Diodes_UDFN-10_1.0x2.5mm_P0.5mm, symbol Power_Protection:D3V3XA4B10LP
- added C1: 2.2uF, symbol Device:C
- added C14, C2: 1uF, symbol Device:C
- added C19, C25, C26, C31: 2u2, symbol Device:C
- added C20, C21, C22, C23, C24, C30, C4: 100n, symbol Device:C
- added C27, C28, C7: 10p, symbol Device:C
- added C29, C6: 10n, symbol Device:C
- added C3: 0.1uF, symbol Device:C
- added C5: 4u7, symbol Device:C
- added C8: 1u, symbol Device:C
- added C9: 22u, symbol Device:C
- added D1: PMEG4010BEA,115, PMEG4010BEA,:SOD2512X110N, symbol PMEG4010BEA,:PMEG4010BEA,115
- added IC1: MS561101BA03-50, MS561101BA03-50, symbol MS561101BA03-50:MS561101BA03-50
- added J1: USB_C_Receptacle_USB2.0_16P, 2171790001(1):MOLEX_2171790001, symbol Connector:USB_C_Receptacle_USB2.0_16P
- added J2: 53254-0470, 532540470, symbol 53254-0470:53254-0470
- added J3: Conn_ARM_JTAG_SWD_10, FTSH-105-01-F-DH:FTSH-105-XX-YYY-DH, symbol Connector:Conn_ARM_JTAG_SWD_10
- added J4: SM08B-SRSS-TB, SM08B-SRSS-TB:JST_SM08B-SRSS-TB, symbol SM08B-SRSS-TB:SM08B-SRSS-TB
- added L1: 2u2, symbol Device:L
- added LED1, LED2, LED3, LED4: SML-P11UTT86R, KDZLV100, symbol RED LED 0402:SML-P11UTT86R
- added R10: 18.2k, symbol Device:R
- added R11, R16, R17: 100k, symbol Device:R
- added R12: 182k, symbol Device:R
- added R13: 1M, symbol Device:R
- added R14, R15, R7, R8: 1k, symbol Device:R
- added R2: 5.1k, symbol Device:R
- added R4, R6, R9: 10k, symbol Device:R
- added R5: 0R, symbol Device:R
- added SW1: PTS810 SJK 250 SMTR LFS, PTS810_CNK, symbol PTS810SJK250SMTR LFS:PTS810_SJK_250_SMTR_LFS
- added U1: TLV76733DRVR, TLV76733DRVR:DRV0006A-IPC_B, symbol TLV76733DRVR:TLV76733DRVR
- added U2: ICM-42688-P, ICM-42688-P:PQFN50P300X250X97-14N, symbol ICM-42688-P:ICM-42688-P
- added U3: STM32F405RGTx, Package_QFP:LQFP-64_10x10mm_P0.5mm, symbol MCU_ST_STM32F4:STM32F405RGTx
- added U4: NUF2042XV6T1G, NUF2042XV6T1G:SON_2XV6T1G_ONS, symbol Power_Protection:USBLC6-2SC6
- added U5: LT8609SIV_TRPBF, LT8609SIV_TRPBF:REG_LT8609SIV_TRPBF, symbol LT8609SIV:LT8609SIV_TRPBF
- added Y1: Crystal, ECS-400-10-37B2-CKM-TR:ECS4001037B2CKMTR, symbol Device:Crystal
- R1: footprint Res 5.1k 0603:RESC1608X55N -> (none)
- R3: value 5.1k -> 10k; footprint Res 5.1k 0603:RESC1608X55N -> (none)
Connections:
- net +3V3: now also R3.1, C1.1, C19.1, C20.1, C21.1, C22.1, C23.1, C24.1, C29.1, C30.1, C31.1, C4.1, IC1.1 (VDD), IC1.2 (PS), J3.1 (VTref), LED2. (A), R16.1, R6.1, R9.1, SW1.1, SW1.2, U1.1 (OUT), U1.2 (SNS), U2.4 (INT1/INT), U2.5 (VDDIO), U2.8 (VDD), U3.1 (VBAT), U3.13 (VDDA), U3.19 (VDD), U3.32 (VDD), U3.48 (VDD), U3.64 (VDD)
- net GND: now also C1.2, C14.2, C19.2, C2.2, C20.2, C21.2, C22.2, C23.2, C24.2, C25.2, C26.2, C27.2, C28.2, C29.2, C3.2, C30.2, C31.2, C4.2, C5.2, C6.2, C8.2, C9.2, IC1.3 (GND), IC1.4 (CSB_1), IC1.5 (CSB_2), J1.A1 (GND), J1.A12 (GND), J1.B1 (GND), J1.B12 (GND), J1.S1 (SHIELD), J2.1, J3.3 (GND), J3.5 (GND), J3.9 (GNDDetect), J4.8, R10.2, R12.2, R14.2, R15.2, R17.2, R2.2, R4.2, R7.2, R8.2, U1.3 (GND), U1.5 (GND), U1.7 (Pad), U2.11 (RESV_11), U2.6 (GND), U2.7 (RESV_7), U2.9 (INT2/FSYNC/CLKIN), U3.12 (VSSA), U3.18 (VSS), U3.63 (VSS), U4.2 (GND), U5.14 (GND), U5.17 (GND), U5.3 (GND), U5.4 (GND), U5.8 (GND); no longer R3.2
- net at R1.1: now also J1.B5 (CC2)
- new net: LED4. (A), R15.1
- new net: C7.1, R12.1, R13.2, U5.13 (FB)
- new net: C28.1, R5.1, Y1.2
- new net: LED3. (A), R14.1
- new net: LED2. (A), R8.1
- new net: L1.1, U5.5 (SW), U5.6 (SW)
- new net: J1.A5 (CC1), R2.1
- new net: C6.1, U5.15 (TR/SS)
- new net: R11.2, U5.12 (PG)
- new net: R10.1, U5.1 (RT)
- new net: C8.1, U5.2 (INTVCC)
- new net: U5.7 (N/C), U5.NC1 (N/C), U5.NC2 (N/C), U5.NC3 (N/C), U5.NC4 (N/C)
- new net: LED1. (A), R7.1
- new net +5V: C2.1, C7.2, C9.1, D1.1 (K), J2.4, L1.2, LED1. (A), R11.1, R13.1, U1.4 (EN), U1.6 (IN), U4.5 (VBUS)
- new net BOOT0: R4.1, SW1.3, SW1.4, U3.60 (BOOT0)
- new net CURR_IN: J4.2, U3.8 (PC0)
- new net D+: J1.A6 (D+), J1.B6 (D+), U3.45 (PA12), U4.3 (I/O2), U4.4 (I/O2)
- new net D-: J1.A7 (D-), J1.B7 (D-), U3.44 (PA11), U4.1 (I/O1), U4.6 (I/O1)
- new net ESC_TLM: J4.1, U3.53 (PC12)
- new net I2C2_SCL: R3.2, U3.29 (PB10)
- new net I2C2_SDA: R6.2, U3.30 (PB11)
- new net LED_OUT: LED4. (A), U3.9 (PC1)
- new net M1: J4.6, U3.37 (PC6)
- new net M2: J4.5, U3.38 (PC7)
- new net M3: J4.4, U3.26 (PB0)
- new net M4: J4.3, U3.27 (PB1)
- new net NRST: C14.1, J3.10 (~{RESET}), R9.2
- new net NRTS: U3.7 (NRST)
- new net OSC_IN: C27.1, U3.5 (PH0), Y1.1
- new net OSC_OUT: R5.2, U3.6 (PH1)
- new net SCL: IC1.8 (SCLK)
- new net SDA: IC1.7 (SDI/SDA)
- new net SPI1_MISO: U2.1 (AP_SDO/AP_AD0), U3.22 (PA6)
- new net SPI1_MOSI: U2.14 (AP_SDA/AP_SDIO/AP_SDI), U3.23 (PA7)
- new net SPI1_NSS: U2.12 (AP_CS), U3.20 (PA4)
- new net SPI1_SCK: U2.13 (AP_SCL/AP_SCLK), U3.21 (PA5)
- new net SWCLK: J3.4 (SWCLK/TCK), R17.1, U3.49 (PA14)
- new net SWDIO: J3.2 (SWDIO/TMS), R16.2, U3.46 (PA13)
- new net SWO: J3.6 (SWO/TDO), U3.55 (PB3)
- new net UART4_RX: J2.3, U3.15 (PA1)
- new net UART4_TX: J2.2, U3.14 (PA0)
- new net VBAT: C5.1, LED3. (A), U5.10 (VIN), U5.11 (EN/UV), U5.9 (VIN)
- new net VBUS: C3.1, D1.2 (A), J1.A4 (VBUS), J1.A9 (VBUS), J1.B4 (VBUS), J1.B9 (VBUS)
- new net VCAP1: C25.1, U3.31 (VCAP_1)
- new net VCAP2: C26.1, U3.47 (VCAP_2)
- new net Vbat: J4.7
- no-connect marks 61 -> 6
Other:
- note added: "Antenna Connector"
- note added: "BUTTONS"
- note added: "Barometer Sensor"
- note added: "Connector"
- note added: "Crystal Oscillator"
- note added: "Current Signal"
- note added: "DSHOT"
- note added: "Decoupling capacitor bank MCU"
- note added: "ESC Connector"
- note added: "GND"
- note added: "IMU 6-Axis Sensor"
- note added: "JTAG - connector"
- note added: "LDO - Voltage Regulator MCU"
- note added: "LED Debugger"
- note added: "Power"
- note added: "STM32F405"
- note added: "Sensor"
- note added: "Step-Down Regulator"
- note added: "Telemetry (UART TX)"
- note added: "USB C + ESD Protection"
- note added: "Vbat"
- note removed: "Auto Programmer"
- note removed: "BOOT"
- note removed: "DECOUPLING"
- note removed: "Debugging LED"
- note removed: "ESD Protection"
- note removed: "ESP32-S3-MINI-1U-N8"
- note removed: "LDO"
- note removed: "RESET"
- note removed: "USB Type-C"
- note removed: "USB-UART Bridge"
