File: Hardware-Electronics/module/Flight-Controller/drone-v0/drone-v0.kicad_sch (KiCad schematic)
At the start: 58 parts, among them IC1 MS561101BA03-50, J1 USB_C_Receptacle_USB2.0_16P, J2 53254-0470, J3 Conn_ARM_JTAG_SWD_10, J4 SM08B-SRSS-TB, SW1 PTS810 SJK 250 SMTR LFS, U1 TLV76733DRVR, U2 ICM-42688-P, U3 STM32F405RGTx, U4 NUF2042XV6T1G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

Commit message: Created initla board outline
Parts:
- removed J2: 53254-0470, 532540470, symbol 53254-0470:53254-0470
- removed LED1, LED2, LED3, LED4: SML-P11UTT86R, KDZLV100, symbol RED LED 0402:SML-P11UTT86R
- removed R5: 0R, symbol Device:R
- removed SW1: PTS810 SJK 250 SMTR LFS, PTS810_CNK, symbol PTS810SJK250SMTR LFS:PTS810_SJK_250_SMTR_LFS
- removed U1: TLV76733DRVR, TLV76733DRVR:DRV0006A-IPC_B, symbol TLV76733DRVR:TLV76733DRVR
- added D2, D3, D4, D5: LED, Red LED 0603:LEDC1608X115N, symbol Device:LED
- added J5: SM04B-SRSS-TB, SM04B-SRSS-TB:CONN_SM04B-SRSS-TB_JST, symbol SM04B-SRSS-TB:SM04B-SRSS-TB
- added R18: 0, Resistor_SMD:R_0603_1608Metric, symbol Device:R
- added SW2: SW_Push, PTS810SJK250SMTRLFS:PTS810SJG250SMTRLFS, symbol Switch:SW_Push
- added U6: TLV76733DRVR, TLV76733DRVR V1:SON65P200X200X80-7N, symbol TLV76733DRVR V1:TLV76733DRVR
- C1, C14, C19, C2, C20, C21, C22, C23, C24, C25, C26, C27, C28, C29, C3, C30, C31, C4, C5, C6, C7, C8, C9: footprint (none) -> Capacitor_SMD:C_0603_1608Metric
- IC1: footprint MS561101BA03-50 -> MS561101BA03-50:MS561101BA03-50
- J1: footprint 2171790001(1):MOLEX_2171790001 -> 217179-0001:2171790001_MOL
- J3: footprint FTSH-105-01-F-DH:FTSH-105-XX-YYY-DH -> 6270XX21721:62701021721
- L1: footprint (none) -> 74438357022:74438357100
- R1, R10, R11, R12, R13, R14, R15, R16, R17, R2, R3, R4, R6, R7, R8, R9: footprint (none) -> Resistor_SMD:R_0603_1608Metric
Connections:
- net NRTS is gone; now on net SWD_NRST: U3.7 (NRST)
- net SCL is gone; now on net I2C2_SCL: IC1.8 (SCLK)
- net SDA is gone; now on net I2C2_SDA: IC1.7 (SDI/SDA)
- net Vbat is gone; now on net VBAT: J4.7
- net +3V3: now also D3.2 (A), R18.2, SW2.2, U6.1 (OUT), U6.2 (SNS); no longer U2.4 (INT1/INT)
- net +5V: now also D2.2 (A), J5.1, U6.4 (EN), U6.6 (IN)
- net BOOT0: now also SW2.1
- net GND: now also J1.A1B12 (GND), J1.B1A12 (GND), J5.4, U6.3 (GND-1), U6.5 (GND); no longer J1.A1 (GND)
- net LED_OUT: now also D4.2 (A)
- net OSC_OUT: now also C28.1, Y1.2
- net UART4_RX: now also J5.2
- net UART4_TX: now also J5.3
- net VBAT: now also D5.2 (A)
- net VBUS: now also J1.A4B9 (VBUS), J1.B4A9 (VBUS); no longer J1.A4 (VBUS)
- net at R15.1: now also D3.1 (K)
- net at R14.1: now also D4.1 (K)
- net at R8.1: now also D5.1 (K)
- net at R7.1: now also D2.1 (K)
- net D+ renamed USB_D+
- net D- renamed USB_D-
- net NRST renamed SWD_NRST
- net SWCLK renamed SWD_CLK
- net SWDIO renamed SWD_IO
- net SWO renamed SWD_TRC
- new net: R18.1, U2.4 (INT1/INT)
- no-connect marks 7 -> 38
Other:
- note added: "LDO - Voltage Regulator"
- note added: "Power Labels"
- note removed: "Current Signal"
- note removed: "DSHOT"
- note removed: "Decoupling capacitor bank MCU"
- note removed: "GND"
- note removed: "LDO - Voltage Regulator MCU"
- note removed: "Telemetry (UART TX)"
- note removed: "Vbat"
- moved on the sheet: C1, C19, C2, C20, C21, C22, C23, C24, C25, C26, C27, C28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
