File: Hardware-Electronics/module/Flight-Controller/drone-v0/drone-v0.kicad_pcb (KiCad board)
At the start: 2 copper layers, 60 x 59.5 mm, 27 parts, among them IC1 REG1117-3.3, IC2 CP2102N-A02-GQFN28, IC3 SBC846BDW1T1G, J2 USB_C_Receptacle_USB2.0_16P, U1 ESP32-S3-MINI-1U-N8, U2 D3V3XA4B10LP

Commit message: Added: STM32 Try resolve with rebase
Parts:
- removed C1, C8: 10uF, Cap 10uF 0603:CAPC1608X90N
- removed C10, C3, C6, C7, C9: 0.1uF, Cap 0.1uF 0603:CAPC1608X90N
- removed C2: 10uF, Cap 0.1uF 0603:CAPC1608X90N
- removed C4, C5: 4.7uF, Cap 4.7uF 0603:CAPC1608X90N
- removed IC1: REG1117-3.3, REG1117-3.3:SOT230P700X180-4N
- removed IC2: CP2102N-A02-GQFN28, CP2102N-A02-GQFN28:QFN50P500X500X80-29N-D
- removed IC3: SBC846BDW1T1G, Res 10k 0603:RESC1608X50N
- removed J2: USB_C_Receptacle_USB2.0_16P, 2171790001(1):MOLEX_2171790001
- removed LED1, LED2: 150060RS83000, Red LED 0603:LEDC1608X115N
- removed R1, R3: 5.1k, Res 5.1k 0603:RESC1608X55N
- removed R2, R7: 1k, Res 1k 0603:RESC1608X50N
- removed R4, R5, R6: 10k, Res 10k 0603:RESC1608X50N
- removed S1, S2: TL3301AF160QG, TL3301AF160QG:TL3301AF160QG
- removed U1: ESP32-S3-MINI-1U-N8, ESP32-S3-MINI-1U-N8:XCVR_ESP32-S3-MINI-1U-N8
- removed U2: D3V3XA4B10LP, Package_DFN_QFN:Diodes_UDFN-10_1.0x2.5mm_P0.5mm
Routing:
- net +5V_USB: track 10.2 -> 0.00 mm, vias 1 -> 0
- net /USB_N: track 2.69 -> 0.00 mm
- net /USB_P: track 2.69 -> 0.00 mm
Other:
- board outline removed

Commit message: Created initla board outline
Parts:
- added C1: 2.2uF, Capacitor_SMD:C_0603_1608Metric, F.Cu at (280.2, 240.1)
- added C14: 1uF, Capacitor_SMD:C_0603_1608Metric, F.Cu at (284.3, 245.1)
- added C19: 2u2, Capacitor_SMD:C_0603_1608Metric, B.Cu at (241.8, 248.2)
- added C2: 1uF, Capacitor_SMD:C_0603_1608Metric, F.Cu at (280.2, 242.6)
- added C20: 100n, Capacitor_SMD:C_0603_1608Metric, B.Cu at (238.4, 248.2)
- added C21: 100n, Capacitor_SMD:C_0603_1608Metric, B.Cu at (233.2, 252.8)
- added C22: 100n, Capacitor_SMD:C_0603_1608Metric, B.Cu at (232.0, 260.2)
- added C23: 100n, Capacitor_SMD:C_0603_1608Metric, B.Cu at (248.4, 255.8)
- added C24: 100n, Capacitor_SMD:C_0603_1608Metric, B.Cu at (248.4, 258.8)
- added C25: 2u2, Capacitor_SMD:C_0603_1608Metric, F.Cu at (288.3, 245.1)
- added C26: 2u2, Capacitor_SMD:C_0603_1608Metric, F.Cu at (288.3, 247.6)
- added C27: 10p, Capacitor_SMD:C_0603_1608Metric, F.Cu at (235.2, 248.2)
- added C28: 10p, Capacitor_SMD:C_0603_1608Metric, F.Cu at (233.0, 250.4)
- added C29: 10n, Capacitor_SMD:C_0603_1608Metric, F.Cu at (259.9, 293.1)
- added C3: 0.1uF, Capacitor_SMD:C_0603_1608Metric, B.Cu at (250.8, 273.6)
- added C30: 100n, Capacitor_SMD:C_0603_1608Metric, F.Cu at (263.0, 296.9)
- added C31: 2u2, Capacitor_SMD:C_0603_1608Metric, F.Cu at (260.4, 296.7)
- added C4: 100n, Capacitor_SMD:C_0603_1608Metric, F.Cu at (256.3, 304.6)
- added C5: 4u7, Capacitor_SMD:C_0603_1608Metric, F.Cu at (280.2, 250.1)
- added C6: 10n, Capacitor_SMD:C_0603_1608Metric, F.Cu at (280.2, 252.6)
- added C7: 10p, Capacitor_SMD:C_0603_1608Metric, F.Cu at (280.2, 255.1)
- added C8: 1u, Capacitor_SMD:C_0603_1608Metric, F.Cu at (284.3, 240.1)
- added C9: 22u, Capacitor_SMD:C_0603_1608Metric, F.Cu at (284.3, 242.6)
- added D1: PMEG4010BEA,115, PMEG4010BEA,:SOD2512X110N, B.Cu at (248.6, 273.2)
- added D2: LED, Red LED 0603:LEDC1608X115N, F.Cu at (294.9, 270.8)
- added D3: LED, Red LED 0603:LEDC1608X115N, F.Cu at (294.9, 273.7)
- added D4: LED, Red LED 0603:LEDC1608X115N, F.Cu at (294.9, 276.7)
- added D5: LED, Red LED 0603:LEDC1608X115N, F.Cu at (294.9, 279.6)
- added IC1: MS561101BA03-50, MS561101BA03-50:MS561101BA03-50, F.Cu at (260.1, 304.5)
- added J1: USB_C_Receptacle_USB2.0_16P, 217179-0001:2171790001_MOL, F.Cu at (240.1, 275.0)
- added J3: Conn_ARM_JTAG_SWD_10, 6270XX21721:62701021721, F.Cu at (257.6, 256.6)
- added J4: SM08B-SRSS-TB, SM08B-SRSS-TB:JST_SM08B-SRSS-TB, F.Cu at (239.6, 237.4)
- added J5: SM04B-SRSS-TB, SM04B-SRSS-TB:CONN_SM04B-SRSS-TB_JST, F.Cu at (222.8, 256.6)
- added L1: 2u2, 74438357022:74438357100, F.Cu at (282.4, 274.4)
- added R1: 5.1k, Resistor_SMD:R_0603_1608Metric, B.Cu at (243.8, 269.6)
- added R10: 18.2k, Resistor_SMD:R_0603_1608Metric, F.Cu at (296.3, 250.1)
- added R11: 100k, Resistor_SMD:R_0603_1608Metric, F.Cu at (296.3, 252.6)
- added R12: 182k, Resistor_SMD:R_0603_1608Metric, F.Cu at (296.3, 255.1)
- added R13: 1M, Resistor_SMD:R_0603_1608Metric, F.Cu at (300.3, 240.1)
- added R14: 1k, Resistor_SMD:R_0603_1608Metric, F.Cu at (300.3, 242.6)
- added R15: 1k, Resistor_SMD:R_0603_1608Metric, F.Cu at (300.3, 245.1)
- added R16: 100k, Resistor_SMD:R_0603_1608Metric, B.Cu at (257.0, 254.0)
- added R17: 100k, Resistor_SMD:R_0603_1608Metric, B.Cu at (257.0, 256.0)
- added R18: 0, Resistor_SMD:R_0603_1608Metric, F.Cu at (261.9, 291.2)
- added R2: 5.1k, Resistor_SMD:R_0603_1608Metric, B.Cu at (236.4, 269.6)
- added R3: 10k, Resistor_SMD:R_0603_1608Metric, F.Cu at (267.2, 301.6)
- added R4: 10k, Resistor_SMD:R_0603_1608Metric, F.Cu at (292.3, 252.6)
- added R6: 10k, Resistor_SMD:R_0603_1608Metric, F.Cu at (267.2, 304.9)
- added R7: 1k, Resistor_SMD:R_0603_1608Metric, F.Cu at (296.3, 242.6)
- added R8: 1k, Resistor_SMD:R_0603_1608Metric, F.Cu at (296.3, 245.1)
- added R9: 10k, Resistor_SMD:R_0603_1608Metric, F.Cu at (296.3, 247.6)
- added SW2: SW_Push, PTS810SJK250SMTRLFS:PTS810SJG250SMTRLFS, F.Cu at (307.0, 249.0)
- added U2: ICM-42688-P, ICM-42688-P:PQFN50P300X250X97-14N, F.Cu at (263.0, 294.0)
- added U3: STM32F405RGTx, Package_QFP:LQFP-64_10x10mm_P0.5mm, F.Cu at (240.0, 257.0)
- added U4: NUF2042XV6T1G, NUF2042XV6T1G:SON_2XV6T1G_ONS, F.Cu at (240.0, 268.4)
- added U5: LT8609SIV_TRPBF, LT8609SIV_TRPBF:REG_LT8609SIV_TRPBF, F.Cu at (275.6, 265.8)
- added U6: TLV76733DRVR, TLV76733DRVR V1:SON65P200X200X80-7N, F.Cu at (304.9, 253.9)
- added Y1: Crystal, ECS-400-10-37B2-CKM-TR:ECS4001037B2CKMTR, F.Cu at (232.2, 247.4)
Other:
- board outline added: 40 x 40 mm
- copper layers 2 -> 4
- rule pad_to_mask_clearance: 0 -> 0.8
