File: Hardware-Electronics/module/ESC/ESC-module.kicad_pcb (KiCad board)
At the start: 4 copper layers, 32.2 x 47.2 mm, 64 parts, among them J1 Conn_01x01, J2 Conn_01x01, J3 Conn_01x01, J4 Conn_01x01, J5 Conn_01x01, J6 Conn_01x06_Pin, J7 Conn_01x02_Pin, J8 Conn_01x02_Pin, Q1 IAUCN04S7N030, Q2 IAUCN04S7N030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

Commit message: Finishing touches
Parts:
- removed D1: D, Diode_SMD:D_0805_2012Metric
- removed J6: Conn_01x06_Pin, Connector_JST:JST_GH_SM06B-GHS-TB_1x06-1MP_P1.25mm_Horizontal
- removed J7: Conn_01x02_Pin, Connector_JST:JST_GH_BM02B-GHS-TBT_1x02-1MP_P1.25mm_Vertical
- added C22: 10u, Capacitor_SMD:C_0805_2012Metric_Pad1.18x1.45mm_HandSolder, F.Cu at (133.2, 88.8)
- added J10: Conn_01x02, Connector_PinSocket_2.54mm:PinSocket_1x02_P2.54mm_Vertical, F.Cu at (154.6, 77.3)
- added J11: Conn_01x01, Connector_Wire:SolderWire-1.5sqmm_1x01_D1.7mm_OD3.9mm, F.Cu at (149.0, 89.9)
- added J12: Conn_01x01, Connector_Wire:SolderWire-1.5sqmm_1x01_D1.7mm_OD3.9mm, F.Cu at (132.8, 72.5)
- added J9: Conn_01x01, Connector_Wire:SolderWire-1.5sqmm_1x01_D1.7mm_OD3.9mm, F.Cu at (149.0, 84.0)
- added JP1: Jumper_2_Open, TestPoint:TestPoint_2Pads_Pitch2.54mm_Drill0.8mm, F.Cu at (131.0, 79.0)
- added JP2: Jumper_2_Open, TestPoint:TestPoint_2Pads_Pitch2.54mm_Drill0.8mm, F.Cu at (154.1, 87.2)
- added R26: 10k, Resistor_SMD:R_0603_1608Metric, F.Cu at (154.2, 90.1)
- added R27: 10k, Resistor_SMD:R_0603_1608Metric, F.Cu at (154.2, 92.6)
- J8: value Conn_01x02_Pin -> Conn_01x01; footprint Connector_JST:JST_GH_BM02B-GHS-TBT_1x02-1MP_P1.25mm_Vertical -> Connector_Wire:SolderWire-1.5sqmm_1x01_D1.7mm_OD3.9mm
- L1: footprint Inductors:IND_BOURNS_SRN3015 -> IND_BOURNS_SRN3015:IND_BOURNS_SRN3015
- R25: value 100k -> 39k
- moved J8 16.7 mm to (149.0, 78.0), turned to 0 degrees
- moved U1 2.25 mm to (130.1, 95.2)
Connections:
- net +15V renamed VM
- J8 pad 1: /PA2 -> GND
- U1 pad 39: unconnected-(U1A-PA15-Pad39) -> /PA15
