File: Hardware-Electronics/module/ESC/ESC-module.kicad_sch (KiCad schematic)
At the start: 66 parts, among them J1 Conn_01x01, J2 Conn_01x01, J3 Conn_01x01, J4 Conn_01x01, J5 Conn_01x01, J6 Conn_01x06_Pin, J7 Conn_01x02_Pin, J8 Conn_01x02_Pin, Q1 IAUCN04S7N030, Q2 IAUCN04S7N030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

Commit message: Finishing touches
Parts:
- removed D1: D, Diode_SMD:D_0805_2012Metric, symbol Device:D
- removed J6: Conn_01x06_Pin, Connector_JST:JST_GH_SM06B-GHS-TB_1x06-1MP_P1.25mm_Horizontal, symbol Connector:Conn_01x06_Pin
- removed J7, J8: Conn_01x02_Pin, Connector_JST:JST_GH_BM02B-GHS-TBT_1x02-1MP_P1.25mm_Vertical, symbol Connector:Conn_01x02_Pin
- added C22: 10u, Capacitor_SMD:C_0805_2012Metric_Pad1.18x1.45mm_HandSolder, symbol Device:C
- added D1: D, symbol STPS0560Z_edit:D
- added J10: Conn_01x02, Connector_PinSocket_2.54mm:PinSocket_1x02_P2.54mm_Vertical, symbol Connector_Generic:Conn_01x02
- added J11, J12, J8, J9: Conn_01x01, Connector_Wire:SolderWire-1.5sqmm_1x01_D1.7mm_OD3.9mm, symbol Connector_Generic:Conn_01x01
- added J6: Conn_ARM_JTAG_SWD_10, symbol Connector:Conn_ARM_JTAG_SWD_10
- added JP1, JP2: Jumper_2_Open, TestPoint:TestPoint_2Pads_Pitch2.54mm_Drill0.8mm, symbol Jumper:Jumper_2_Open
- added R26, R27: 10k, Resistor_SMD:R_0603_1608Metric, symbol Device:R
- L1: footprint Inductors:IND_BOURNS_SRN3015 -> IND_BOURNS_SRN3015:IND_BOURNS_SRN3015
- R25: value 100k -> 39k
Connections:
- net BOOT: now also JP1.2 (B), R26.2
- net GND: now also C22.2, D1.2 (A), J6.3 (GND), J6.5 (GND), J6.9 (GNDDetect), J8.1 (Pin_1), R26.1, R27.1
- net NRST: now also J6.10 (~{RESET}), JP2.1 (A)
- net PA2: now also J9.1 (Pin_1)
- net PB6: now also J10.2 (Pin_2)
- net PB7: now also J10.1 (Pin_1)
- net SWDCLK: now also J11.1 (Pin_1), J6.4 (SWCLK/TCK)
- net SWDIO: now also J6.2 (SWDIO/TMS)
- net VDD: now also J6.1 (VTref), JP1.1 (A)
- net at L1.2, U1.9 (SW): now also D1.1 (K)
- net PA15: now reaches U1.39 (PA15)
- net PA15: now also J12.1 (Pin_1)
- net +15V renamed VM
- net VM: now also C22.1
- new net: JP2.2 (B), R27.2
- no-connect marks 5 -> 6
Other:
- note added: "Battery in"
- note added: "Bootloader enable"
- note added: "Emergency reset"
- note added: "RX"
- note added: "TX"
- note added: "USART2"
- note added: "USART_1"
- note removed: "6-step sensor-less"
- note removed: "Debug/UART"
- moved on the sheet: C10, C11, C12, C13, C14, C15, C16, C17, C18, C19, C20, C21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

Commit message: Forgot footprint for SWD
Parts:
- J6: footprint (none) -> footprints:SAMTEC_FTSH-105-01-F-DH
Changed lines of the file:
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@@
 			)
 		)
-		(property "Footprint" ""
+		(property "Footprint" "footprints:SAMTEC_FTSH-105-01-F-DH"
 			(at 53.34 247.65 0)
 			(effects
